File: kicad/sharpkey.kicad_sch (KiCad schematic)
At the start: 41 parts, among them J1 Host I/F, J2 PS/2 Keyboard, J3 PGM/OLED, Q1 MMDT3904, SW1 WiFi EN, U1 AMS1117-3.3, U2 74LS257, U3 ESP32-S AI Thinker

Commit message: Schematic updates and docs
Parts:
- R21: value DNP -> 10K
Other:
- note added: "DSCK / DSDA - I2C Interface to an OLED Display. RXD/TXD. - UART Receive and Transmit. DTR/RTS - UART control lines used for programming and reset of the ESP32."
- note added: "MZ-2500/2800 Signal Key 2 KD0 - 3 KD1 - 4 KD2 - 5 KD3 - Bi-directional Bus 6 KD4 - H:Key Data, L:Strobe All Data 7 MPX - H:Upper Nibble, L:Lower Nibble 8 ~{RTSN} - H:Row Sent, L:Key Data Returned"
- note added: "Mouse Signal Key 2 - 3 MSCTRL - Mouse Control Clock 4 MSDATA - Mouse Data 5 - 6 - 7 - 8 -"
- note added: "X1 Signal Key 2 - 3 DATA - X1 Key Data 4 - 5 - 6 - 7 - 8 -"
- note added: "X68000 Keyboard Signal Key 2 - 3 TXD - Transmit Data 4 RXD - Receive Data 5 READY - Keyboard Ready 6 REMOTE - Remote 7 - 8 -"
- note removed: "DSCK / DSDA - I2C Interface to an OLED Display. RXD/TXD. - UART Receive and Transmit. DTR/RTS - UART control lines used for programming and reset of the ESP32. NB: MPX must be strapped low or N/C to program."
- note removed: "MZ-2500/2800 Signal Key 2 ~{RTSN} - H:Row Sent, L:Key Data Returned 3 KD0 - 4 KD1 - 5 KD2 - 6 KD3 - Bi-directional Bus 7 KD4 - H:Key Data, L:Strobe All Data 8 MPX - H:Upper Nibble, L:Lower Nibble"
- note removed: "Mouse Signal Key 2 - N/C (pulled high internally) 3 MSCTRL - Mouse Control Clock 4 MSDATA - Mouse Data 5 - Strap low 6 - Strap low 7 - Strap high 8 - Strap low"
- note removed: "NB: MPX must be strapped low or N/C."
- note removed: "X1 Signal Key 2 - Strap low 3 DATA - X1 Key Data 4 - Strap low 5 - Strap low 6 - Strap low 7 - Strap low 8 - Strap low"
- note removed: "X68000 Keyboard Signal Key 2 - N/C (pulled high internally) 3 TXD - Transmit Data 4 RXD - Receive Data 5 READY - Keyboard Ready 6 REMOTE - Remote 7 - Strap low 8 - Strap low"
Changed lines of the file:
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@@
     (rev "1.3")
     (comment 1 "dedicated to the Host I/F, the second core to PS/2 capture, vector build and map.")
-    (comment 2 "toolchain. The requirements require control down to 100ns so one cpu core is always")
+    (comment 2 "toolchain. The requirements require control down to 100ns so on cpu core is always")
     (comment 3 "This design uses the common ESP32 SoC for its performance, low power and development ")
     (comment 4 "PS/2 to Sharp MZ-2500/MZ-2800/X1/X68K Keyboard Interface.")
@@
     (effects (font (size 1.27 1.27)) (justify left bottom))
   )
-  (text "NB: MPX must be strapped low or N/C." (at 19.05 177.8 0)
-    (effects (font (size 0.7874 0.7874)) (justify left bottom))
-  )
-  (text "     Mouse Signal Key\n\n2          - N/C (pulled high internally)\n3 MSCTRL  - Mouse Control Clock\n4 MSDATA  - Mouse Data\n5          - Strap low\n6          - Strap low\n7          - Strap high\n8          - Strap low"
-    (at 13.97 167.64 0)
+  (text "     Mouse Signal Key\n\n2          - \n3 MSCTRL  - Mouse Control Clock\n4 MSDATA  - Mouse Data\n5          - \n6          - \n7          - \n8          - "
+    (at 19.05 172.72 0)
     (effects (font (size 0.7874 0.7874)) (justify left bottom))
   )
@@
     (effects (font (size 1.27 1.27)) (justify left bottom))
   )
-  (text "DSCK / DSDA - I2C Interface to an OLED Display.\nRXD/TXD.     - UART Receive and Transmit.\nDTR/RTS      - UART control lines used for programming \n                  and reset of the ESP32.\n\nNB: MPX must be strapped low or N/C to program."
-    (at 247.65 80.01 0)
+  (text "DSCK / DSDA - I2C Interface to an OLED Display.\nRXD/TXD.     - UART Receive and Transmit.\nDTR/RTS      - UART control lines used for programming \n                  and reset of the ESP32."
+    (at 247.65 76.2 0)
     (effects (font (size 0.7874 0.7874)) (justify left bottom))
   )
-  (text "     X68000 Keyboard Signal Key\n\n2         - N/C (pulled high internally)\n3 TXD    - Transmit Data\n4 RXD    - Receive Data\n5 READY  - Keyboard Ready\n6 REMOTE - Remote\n7         - Strap low\n8         - Strap low\n"
-    (at 13.97 154.94 0)
+  (text "     X68000 Keyboard Signal Key\n\n2         - \n3 TXD    - Transmit Data\n4 RXD    - Receive Data\n5 READY  - Keyboard Ready\n6 REMOTE - Remote\n7         - \n8         - "
+    (at 19.05 158.75 0)
     (effects (font (size 0.7874 0.7874)) (justify left bottom))
   )
-  (text "     X1 Signal Key\n\n2        - Strap low\n3 DATA   - X1 Key Data\n4        - Strap low\n5        - Strap low\n6        - Strap low\n7        - Strap low\n8        - Strap low"
-    (at 13.97 142.24 0)
+  (text "     X1 Signal Key\n\n2      -\n3 DATA - X1 Key Data\n4      -\n5      - \n6      - \n7      - \n8      - "
+    (at 19.05 144.78 0)
     (effects (font (size 0.7874 0.7874)) (justify left bottom))
   )
-  (text "     MZ-2500/2800 Signal Key\n\n2 ~{RTSN} - H:Row Sent, L:Key Data Returned\n3 KD0  -\n4 KD1  -\n5 KD2  -\n6 KD3  - Bi-directional Bus\n7 KD4  - H:Key Data, L:Strobe All Data\n8 MPX  - H:Upper Nibble, L:Lower Nibble"
-    (at 13.97 129.54 0)
+  (text "     MZ-2500/2800 Signal Key\n\n2 KD0  -\n3 KD1  -\n4 KD2  -\n5 KD3  - Bi-directional Bus\n6 KD4  - H:Key Data, L:Strobe All Data\n7 MPX  - H:Upper Nibble, L:Lower Nibble\n8 ~{RTSN} - H:Row Sent, L:Key Data Returned"
+    (at 19.05 130.81 0)
     (effects (font (size 0.7874 0.7874)) (justify left bottom))
   )
@@
       (effects (font (size 0.7874 0.7874)) (justify left))
     )
-    (property "Value" "DNP" (id 1) (at 143.51 90.17 0)
+    (property "Value" "10K" (id 1) (at 143.51 90.17 0)
       (effects (font (size 0.7874 0.7874)) (justify left))
     )
@@
     )
     (path "/fabcffe5-3ed2-40e2-896a-ed011b2d8803"
-      (reference "R21") (unit 1) (value "DNP") (footprint "Resistor_SMD:R_0805_2012Metric")
+      (reference "R21") (unit 1) (value "10K") (footprint "Resistor_SMD:R_0805_2012Metric")
     )
     (path "/00000000-0000-0000-0000-000062009785"
